Commit message: fix robot shape, add obstacles

File: Add Robot/ws/src/gpu_slam_bot/urdf/gpu_bot.urdf.xacro (robot description, xacro)
@@ -1,65 +1,136 @@
 <?xml version="1.0"?>
-<robot name="gpu_slam_bot" xmlns:xacro="http://ros.org/wiki/xacro">
-  <!-- Main base link -->
+<robot xmlns:xacro="http://www.ros.org/wiki/xacro" name="gpu_slam_bot">
+  <!-- Robot parameters -->
+  <xacro:property name="base_width" value="0.30"/>
+  <xacro:property name="base_length" value="0.45"/>
+  <xacro:property name="base_height" value="0.12"/>
+  <xacro:property name="wheel_radius" value="0.07"/>
+  <xacro:property name="wheel_width" value="0.06"/>
+  <xacro:property name="wheel_separation" value="0.35"/>
+  <!-- Materials -->
+  <material name="base_blue"><color rgba="0 0.5 1 1"/></material>
+  <material name="lidar_red"><color rgba="1 0 0 1"/></material>
+  <material name="wheel_black"><color rgba="0 0 0 1"/></material>
+  <material name="caster_grey"><color rgba="0.4 0.4 0.4 1"/></material>
+  <!-- Base link -->
   <link name="base_link">
     <visual>
-      <geometry>
-        <box size="0.4 0.3 0.1"/>
-      </geometry>
-      <material name="blue"/>
+      <origin xyz="0 0 0" rpy="0 0 0"/>
+      <geometry><box size="${base_length} ${base_width} ${base_height}"/></geometry>
+      <material name="base_blue"/>
     </visual>
     <collision>
-      <geometry>
-        <box size="0.4 0.3 0.1"/>
-      </geometry>
+      <origin xyz="0 0 0" rpy="0 0 0"/>
+      <geometry><box size="${base_length} ${base_width} ${base_height}"/></geometry>
     </collision>
     <inertial>
-      <mass value="5.0"/>
-      <inertia ixx="0.1" iyy="0.1" izz="0.1"/>
+      <origin xyz="0 0 0" rpy="0 0 0"/>
+      <mass value="3.0"/>
+      <inertia ixx="${(1/12)*3*(base_width**2 + base_height**2)}"
+               iyy="${(1/12)*3*(base_length**2 + base_height**2)}"
+               izz="${(1/12)*3*(base_length**2 + base_width**2)}"
+               ixy="0" ixz="0" iyz="0"/>
     </inertial>
   </link>
-  <!-- 4 wheels -->
-  <xacro:macro name="wheel" params="name x y">
-    <link name="${name}">
-      <visual>
-        <geometry>
-          <cylinder length="0.05" radius="0.05"/>
-        </geometry>
-        <material name="black"/>
-      </visual>
-      <collision>
-        <geometry>
-          <cylinder length="0.05" radius="0.05"/>
-        </geometry>
-      </collision>
-      <inertial>
-        <mass value="1.0"/>
-        <inertia ixx="0.01" iyy="0.01" izz="0.01"/>
-      </inertial>
-    </link>
-    <joint name="${name}_joint" type="continuous">
-      <parent link="base_link"/>
-      <child link="${name}"/>
-      <origin xyz="${x} ${y} -0.05" rpy="0 1.5708 0"/>
-      <axis xyz="0 0 1"/>
-    </joint>
-  </xacro:macro>
-  <xacro:wheel name="front_left_wheel"  x="0.15" y="0.15"/>
-  <xacro:wheel name="front_right_wheel" x="0.15" y="-0.15"/>
-  <xacro:wheel name="rear_left_wheel"   x="-0.15" y="0.15"/>
-  <xacro:wheel name="rear_right_wheel"  x="-0.15" y="-0.15"/>
-  <!-- Lidar on top -->
+  <!-- Wheels -->
+  <link name="wheel_left">
+    <visual>
+      <origin xyz="0 0 0" rpy="1.5708 0 0"/>
+      <geometry><cylinder radius="${wheel_radius}" length="${wheel_width}"/></geometry>
+      <material name="wheel_black"/>
+    </visual>
+    <collision>
+      <origin xyz="0 0 0" rpy="1.5708 0 0"/>
+      <geometry><cylinder radius="${wheel_radius}" length="${wheel_width}"/></geometry>
+    </collision>
+    <inertial>
+      <origin xyz="0 0 0" rpy="1.5708 0 0"/>
+      <mass value="0.5"/>
+      <inertia ixx="0.0013" iyy="0.0024" izz="0.0013" ixy="0" ixz="0" iyz="0"/>
+    </inertial>
+  </link>
+  <link name="wheel_right">
+    <visual>
+      <origin xyz="0 0 0" rpy="1.5708 0 0"/>
+      <geometry><cylinder radius="${wheel_radius}" length="${wheel_width}"/></geometry>
+      <material name="wheel_black"/>
+    </visual>
+    <collision>
+      <origin xyz="0 0 0" rpy="1.5708 0 0"/>
+      <geometry><cylinder radius="${wheel_radius}" length="${wheel_width}"/></geometry>
+    </collision>
+    <inertial>
+      <origin xyz="0 0 0" rpy="1.5708 0 0"/>
+      <mass value="0.5"/>
+      <inertia ixx="0.0013" iyy="0.0024" izz="0.0013" ixy="0" ixz="0" iyz="0"/>
+    </inertial>
+  </link>
+  <!-- Wheel joints -->
+  <joint name="wheel_left_joint" type="continuous">
+    <parent link="base_link"/>
+    <child link="wheel_left"/>
+    <origin xyz="0 ${wheel_separation/2} ${-base_height/2 + wheel_radius}" rpy="0 0 0"/>
+    <axis xyz="0 1 0"/>
+  </joint>
+  <joint name="wheel_right_joint" type="continuous">
+    <parent link="base_link"/>
+    <child link="wheel_right"/>
+    <origin xyz="0 ${-wheel_separation/2} ${-base_height/2 + wheel_radius}" rpy="0 0 0"/>
+    <axis xyz="0 1 0"/>
+  </joint>
+  <!-- Wheel transmissions for ROS 2 Control -->
+  <transmission name="left_wheel_trans">
+    <type>transmission_interface/SimpleTransmission</type>
+    <joint name="wheel_left_joint"/>
+    <actuator name="left_motor"/>
+  </transmission>
+  <transmission name="right_wheel_trans">
+    <type>transmission_interface/SimpleTransmission</type>
+    <joint name="wheel_right_joint"/>
+    <actuator name="right_motor"/>
+  </transmission>
+  <!-- Lidar -->
   <link name="lidar_link">
     <visual>
-      <geometry>
-        <cylinder length="0.05" radius="0.05"/>
-      </geometry>
-      <material name="grey"/>
+      <origin xyz="0 0 0.03" rpy="0 0 0"/>
+      <geometry><cylinder length="0.06" radius="0.055"/></geometry>
+      <material name="lidar_red"/>
     </visual>
+    <collision>
+      <origin xyz="0 0 0.03" rpy="0 0 0"/>
+      <geometry><cylinder length="0.06" radius="0.055"/></geometry>
+    </collision>
+    <inertial>
+      <origin xyz="0 0 0.03" rpy="0 0 0"/>
+      <mass value="0.1"/>
+      <inertia ixx="0.0003" iyy="0.0003" izz="0.0002" ixy="0" ixz="0" iyz="0"/>
+    </inertial>
   </link>
   <joint name="lidar_joint" type="fixed">
     <parent link="base_link"/>
     <child link="lidar_link"/>
-    <origin xyz="0 0 0.1"/>
+    <origin xyz="0 0 ${base_height/2 + 0.03}" rpy="0 0 0"/>
+  </joint>
+  <!-- Caster -->
+  <link name="caster_link">
+    <visual>
+      <origin xyz="0 0 0" rpy="0 0 0"/>
+      <geometry><sphere radius="0.03"/></geometry>
+      <material name="caster_grey"/>
+    </visual>
+    <collision>
+      <origin xyz="0 0 0" rpy="0 0 0"/>
+      <geometry><sphere radius="0.03"/></geometry>
+    </collision>
+    <inertial>
+      <origin xyz="0 0 0" rpy="0 0 0"/>
+      <mass value="0.1"/>
+      <inertia ixx="1e-5" iyy="1e-5" izz="1e-5" ixy="0" ixz="0" iyz="0"/>
+    </inertial>
+  </link>
+  <joint name="caster_joint" type="fixed">
+    <parent link="base_link"/>
+    <child link="caster_link"/>
+    <origin xyz="-${base_length/2} 0 ${-base_height/2 + 0.03}" rpy="0 0 0"/>
   </joint>
 </robot>

File: Add Robot/ws/src/gpu_slam_bot/urdf/gpu_slam_bot.urdf.xacro (robot description, xacro)
@@ -1,9 +1,15 @@
 <?xml version="1.0"?>
 <robot xmlns:xacro="http://www.ros.org/wiki/xacro" name="gpu_slam_bot">
-  <!-- convenience materials (named) -->
+  <!-- Robot parameters -->
+  <xacro:property name="base_width" value="0.30"/>
+  <xacro:property name="base_length" value="0.45"/>
+  <xacro:property name="base_height" value="0.12"/>
+  <xacro:property name="wheel_radius" value="0.07"/>
+  <xacro:property name="wheel_width" value="0.06"/>
+  <xacro:property name="wheel_separation" value="0.35"/>
+  <!-- convenience materials -->
   <material name="base_blue"><color rgba="0 0.5 1 1"/></material>
   <material name="lidar_red"><color rgba="1 0 0 1"/></material>
   <material name="wheel_black"><color rgba="0 0 0 1"/></material>
-  <material name="arrow_red"><color rgba="1 0 0 1"/></material>
   <material name="caster_grey"><color rgba="0.4 0.4 0.4 1"/></material>
   <!-- base -->
@@ -11,14 +17,18 @@
     <visual>
       <origin xyz="0 0 0" rpy="0 0 0"/>
-      <geometry><box size="0.45 0.30 0.12"/></geometry>
+      <geometry><box size="${base_length} ${base_width} ${base_height}"/></geometry>
       <material name="base_blue"/>
     </visual>
     <collision>
       <origin xyz="0 0 0" rpy="0 0 0"/>
-      <geometry><box size="0.45 0.30 0.12"/></geometry>
+      <geometry><box size="${base_length} ${base_width} ${base_height}"/></geometry>
     </collision>
     <inertial>
+      <origin xyz="0 0 0" rpy="0 0 0"/>
       <mass value="3.0"/>
-      <inertia ixx="0.02" iyy="0.02" izz="0.02" ixy="0" ixz="0" iyz="0"/>
+      <inertia ixx="${(1/12) * 3.0 * (base_width*base_width + base_height*base_height)}"
+               iyy="${(1/12) * 3.0 * (base_length*base_length + base_height*base_height)}"
+               izz="${(1/12) * 3.0 * (base_length*base_length + base_width*base_width)}"
+               ixy="0" ixz="0" iyz="0"/>
     </inertial>
   </link>
@@ -26,15 +36,16 @@
   <link name="lidar_link">
     <visual>
-      <origin xyz="0 0 0.09" rpy="0 0 0"/>
+      <origin xyz="0 0 0.03" rpy="0 0 0"/>
       <geometry><cylinder length="0.06" radius="0.055"/></geometry>
       <material name="lidar_red"/>
     </visual>
     <collision>
-      <origin xyz="0 0 0.09" rpy="0 0 0"/>
+      <origin xyz="0 0 0.03" rpy="0 0 0"/>
       <geometry><cylinder length="0.06" radius="0.055"/></geometry>
     </collision>
     <inertial>
+      <origin xyz="0 0 0.03" rpy="0 0 0"/>
       <mass value="0.1"/>
-      <inertia ixx="0.001" iyy="0.001" izz="0.001" ixy="0" ixz="0" iyz="0"/>
+      <inertia ixx="0.0003" iyy="0.0003" izz="0.0002" ixy="0" ixz="0" iyz="0"/>
     </inertial>
   </link>
@@ -42,77 +53,99 @@
     <parent link="base_link"/>
     <child link="lidar_link"/>
-    <origin xyz="0 0 0.12" rpy="0 0 0"/>
+    <origin xyz="0 0 ${base_height/2 + 0.03}" rpy="0 0 0"/>
   </joint>
-  <!-- wheels: left & right (visual rotated so cylinder looks like a wheel) -->
-  <!-- Wheel geometry is defined as cylinder with small length (thickness) and radius -->
+  <!-- wheels -->
   <link name="wheel_left">
     <visual>
-      <!-- rotate cylinder so its axis aligns with joint rotation axis (Y) -->
-      <origin xyz="0 0.175 -0.05" rpy="1.5708 0 0"/>
-      <geometry><cylinder length="0.06" radius="0.07"/></geometry>
+      <origin xyz="0 0 0" rpy="1.5708 0 0"/>
+      <geometry><cylinder length="${wheel_width}" radius="${wheel_radius}"/></geometry>
       <material name="wheel_black"/>
     </visual>
     <collision>
-      <origin xyz="0 0.175 -0.05" rpy="1.5708 0 0"/>
-      <geometry><cylinder length="0.06" radius="0.07"/></geometry>
+      <origin xyz="0 0 0" rpy="1.5708 0 0"/>
+      <geometry><cylinder length="${wheel_width}" radius="${wheel_radius}"/></geometry>
     </collision>
+    <inertial>
+      <origin xyz="0 0 0" rpy="1.5708 0 0"/>
+      <mass value="0.5"/>
+      <inertia ixx="0.0013" iyy="0.0024" izz="0.0013" ixy="0" ixz="0" iyz="0"/>
+    </inertial>
   </link>
   <link name="wheel_right">
     <visual>
-      <origin xyz="0 -0.175 -0.05" rpy="1.5708 0 0"/>
-      <geometry><cylinder length="0.06" radius="0.07"/></geometry>
+      <origin xyz="0 0 0" rpy="1.5708 0 0"/>
+      <geometry><cylinder length="${wheel_width}" radius="${wheel_radius}"/></geometry>
       <material name="wheel_black"/>
     </visual>
     <collision>
-      <origin xyz="0 -0.175 -0.05" rpy="1.5708 0 0"/>
-      <geometry><cylinder length="0.06" radius="0.07"/></geometry>
+      <origin xyz="0 0 0" rpy="1.5708 0 0"/>
+      <geometry><cylinder length="${wheel_width}" radius="${wheel_radius}"/></geometry>
     </collision>
+    <inertial>
+      <origin xyz="0 0 0" rpy="1.5708 0 0"/>
+      <mass value="0.5"/>
+      <inertia ixx="0.0013" iyy="0.0024" izz="0.0013" ixy="0" ixz="0" iyz="0"/>
+    </inertial>
   </link>
+  <!-- wheel joints -->
   <joint name="wheel_left_joint" type="continuous">
     <parent link="base_link"/>
     <child link="wheel_left"/>
-    <!-- joint at the same position as the wheel visual origin (but without the rotation) -->
-    <origin xyz="0 0.175 -0.05" rpy="0 0 0"/>
-    <axis xyz="0 1 0"/> <!-- rotate around robot Y axis (wheel axle) -->
+    <origin xyz="0 ${wheel_separation/2} ${-base_height/2 + wheel_radius}" rpy="0 0 0"/>
+    <axis xyz="0 1 0"/>
   </joint>
   <joint name="wheel_right_joint" type="continuous">
     <parent link="base_link"/>
     <child link="wheel_right"/>
-    <origin xyz="0 -0.175 -0.05" rpy="0 0 0"/>
+    <origin xyz="0 ${-wheel_separation/2} ${-base_height/2 + wheel_radius}" rpy="0 0 0"/>
     <axis xyz="0 1 0"/>
   </joint>
-  <!-- small caster at the back for stability -->
-  <link name="caster">
+  <!-- caster wheel -->
+  <link name="caster_link">
     <visual>
-      <origin xyz="-0.18 0 -0.06" rpy="0 0 0"/>
+      <origin xyz="0 0 0" rpy="0 0 0"/>
       <geometry><sphere radius="0.03"/></geometry>
       <material name="caster_grey"/>
     </visual>
     <collision>
-      <origin xyz="-0.18 0 -0.06" rpy="0 0 0"/>
+      <origin xyz="0 0 0" rpy="0 0 0"/>
       <geometry><sphere radius="0.03"/></geometry>
     </collision>
+    <inertial>
+      <origin xyz="0 0 0" rpy="0 0 0"/>
+      <mass value="0.1"/>
+      <inertia ixx="1e-5" iyy="1e-5" izz="1e-5" ixy="0" ixz="0" iyz="0"/>
+    </inertial>
   </link>
   <joint name="caster_joint" type="fixed">
     <parent link="base_link"/>
-    <child link="caster"/>
-    <origin xyz="-0.18 0 -0.06" rpy="0 0 0"/>
+    <child link="caster_link"/>
+    <origin xyz="-${base_length/2} 0 ${-base_height/2 + 0.03}" rpy="0 0 0"/>
   </joint>
-  <!-- direction arrow (rotated so it points forward along +X) -->
-  <link name="direction_arrow">
-    <visual>
-      <origin xyz="0.18 0 0.06" rpy="0 1.5708 0"/> <!-- rotate so cylinder points along X -->
-      <geometry><cylinder length="0.12" radius="0.02"/></geometry>
-      <material name="arrow_red"/>
-    </visual>
-    <collision>
-      <origin xyz="0.18 0 0.06" rpy="0 1.5708 0"/>
-      <geometry><cylinder length="0.12" radius="0.02"/></geometry>
-    </collision>
-  </link>
-  <joint name="arrow_joint" type="fixed">
-    <parent link="base_link"/>
-    <child link="direction_arrow"/>
-    <origin xyz="0 0 0.07" rpy="0 0 0"/>
-  </joint>
+  <!-- Gazebo plugins -->
+  <gazebo>
+    <plugin name="diff_drive" filename="libgazebo_ros_diff_drive.so">
+      <ros>
+        <namespace>/</namespace>
+        <argument>cmd_vel:=cmd_vel</argument>
+        <argument>odom:=odom</argument>
+      </ros>
+      <update_rate>50</update_rate>
+      <left_joint>wheel_left_joint</left_joint>
+      <right_joint>wheel_right_joint</right_joint>
+      <wheel_separation>${wheel_separation}</wheel_separation>
+      <wheel_diameter>${2*wheel_radius}</wheel_diameter>
+      <publish_odom>true</publish_odom>
+      <publish_wheel_tf>true</publish_wheel_tf>
+      <publish_tf>true</publish_tf>
+    </plugin>
+    <plugin name="lidar_plugin" filename="libgazebo_ros_ray_sensor.so">
+      <ros>
+        <namespace>/</namespace>
+        <argument>scan:=scan</argument>
+      </ros>
+      <update_rate>10</update_rate>
+      <frame_name>lidar_link</frame_name>
+    </plugin>
+  </gazebo>
 </robot>
